File: EAGLE/projects/Kontrol_S4_MK4/potboard.brd (EAGLE design)
At the start: 143 x 51.8 mm, 36 parts, among them IC2 74HC595D, IC3 74HC165D

Commit message: update silkscreen
Parts:
- C1, C2: value (none) -> 0.1u
Routing:
- net D3: track 53.2 -> 58.1 mm
- net D2: track 63.1 -> 60.6 mm
Other:
- board text added: "27 10 21"
- board text removed: "25 11 20"
Changed lines of the file:
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@@
 <?xml version="1.0" encoding="utf-8"?>
 <!DOCTYPE eagle SYSTEM "eagle.dtd">
-<eagle version="9.6.1">
+<eagle version="9.5.2">
 <drawing>
 <settings>
@@
 <wire x1="99" y1="49" x2="99" y2="51.8" width="0" layer="20"/>
 <text x="109" y="45" size="1.016" layer="25">Will Willems</text>
-<text x="109" y="43" size="1.016" layer="25">25 11 20</text>
+<text x="109" y="43" size="1.016" layer="25">27 10 21</text>
 <wire x1="0" y1="7" x2="143" y2="7" width="0.1524" layer="21" style="shortdash"/>
 <text x="18" y="43.5" size="1.016" layer="22" distance="25" rot="MR90" align="bottom-right">1.
@@
 </autorouter>
 <elements>
-<element name="C1" library="adafruit" package="C1206" value="" x="41.9" y="34.3" smashed="yes">
-<attribute name="NAME" x="40.63" y="35.443" size="1.27" layer="25"/>
-<attribute name="VALUE" x="40.63" y="31.887" size="1.27" layer="27"/>
-</element>
-<element name="C2" library="adafruit" package="C1206" value="" x="77" y="47" smashed="yes">
+<element name="C1" library="adafruit" package="C1206" value="0.1u" x="41.9" y="34.3" smashed="yes">
+<attribute name="NAME" x="36.63" y="33.443" size="1.27" layer="25"/>
+<attribute name="VALUE" x="44.63" y="33.887" size="1.27" layer="27"/>
+</element>
+<element name="C2" library="adafruit" package="C1206" value="0.1u" x="77" y="47" smashed="yes">
 <attribute name="NAME" x="75.73" y="48.143" size="1.27" layer="25"/>
 <attribute name="VALUE" x="75.73" y="44.587" size="1.27" layer="27"/>
@@
 </element>
 <element name="IC2" library="74xx-eu" library_urn="urn:adsk.eagle:library:85" package="SO16" package3d_urn="urn:adsk.eagle:package:2010/1" value="74HC595D" x="42" y="41" smashed="yes" rot="R90">
-<attribute name="NAME" x="43.905" y="35.539" size="1.27" layer="25" ratio="10" rot="R180"/>
+<attribute name="NAME" x="45.905" y="48.539" size="1.27" layer="25" ratio="10" rot="R180"/>
 <attribute name="POPULARITY" value="21" x="85.18" y="90.53" size="1.778" layer="27" rot="R90" display="off"/>
 <attribute name="VALUE" x="42.762" y="37.19" size="1.27" layer="27" ratio="10" rot="R90"/>
@@
 </element>
 <element name="R6" library="rcl" library_urn="urn:adsk.eagle:library:334" package="R0805" package3d_urn="urn:adsk.eagle:package:23553/2" value="10K" x="60" y="42.5" smashed="yes">
-<attribute name="NAME" x="59.365" y="43.77" size="1.27" layer="25"/>
+<attribute name="NAME" x="55.365" y="41.77" size="1.27" layer="25"/>
 <attribute name="POPULARITY" value="85" x="91.75" y="-18.46" size="1.778" layer="27" display="off"/>
 <attribute name="SPICEPREFIX" value="R" x="91.75" y="-18.46" size="1.778" layer="27" display="off"/>
-<attribute name="VALUE" x="59.365" y="39.96" size="1.27" layer="27"/>
+<attribute name="VALUE" x="62.365" y="41.96" size="0.6096" layer="27"/>
 </element>
 <element name="R8" library="rcl" library_urn="urn:adsk.eagle:library:334" package="R0805" package3d_urn="urn:adsk.eagle:package:23553/2" value="10K" x="60" y="40" smashed="yes">
-<attribute name="NAME" x="59.365" y="41.27" size="1.27" layer="25"/>
+<attribute name="NAME" x="55.365" y="39.27" size="1.27" layer="25"/>
 <attribute name="POPULARITY" value="85" x="96.83" y="-20.96" size="1.778" layer="27" display="off"/>
 <attribute name="SPICEPREFIX" value="R" x="96.83" y="-20.96" size="1.778" layer="27" display="off"/>
-<attribute name="VALUE" x="59.365" y="37.46" size="1.27" layer="27"/>
+<attribute name="VALUE" x="62.365" y="39.46" size="0.6096" layer="27"/>
 </element>
 <element name="R9" library="rcl" library_urn="urn:adsk.eagle:library:334" package="R0805" package3d_urn="urn:adsk.eagle:package:23553/2" value="10K" x="60" y="37.5" smashed="yes">
-<attribute name="NAME" x="59.365" y="38.77" size="1.27" layer="25"/>
+<attribute name="NAME" x="55.365" y="36.77" size="1.27" layer="25"/>
 <attribute name="POPULARITY" value="85" x="101.91" y="-23.46" size="1.778" layer="27" display="off"/>
 <attribute name="SPICEPREFIX" value="R" x="101.91" y="-23.46" size="1.778" layer="27" display="off"/>
-<attribute name="VALUE" x="59.365" y="34.96" size="1.27" layer="27"/>
+<attribute name="VALUE" x="62.365" y="36.96" size="0.6096" layer="27"/>
 </element>
 <element name="U$1" library="S4" package="BUTTON_S4" value="BUTTON_S4" x="24" y="13" smashed="yes"/>
@@
 <wire x1="60.083190625" y1="10.59993125" x2="60.1218" y2="10.59993125" width="0.4" layer="1"/>
 <wire x1="60.1218" y1="10.59993125" x2="67.62293125" y2="10.59993125" width="0.4" layer="1"/>
-<wire x1="49.949859375" y1="8.99998125" x2="49.9872" y2="8.99998125" width="0.4" layer="1"/>
-<wire x1="49.9872" y1="8.99998125" x2="53.483" y2="8.99998125" width="0.4" layer="1"/>
-<wire x1="53.483" y1="8.99998125" x2="55.08295" y2="10.59993125" width="0.4" layer="1"/>
+<wire x1="55.08295" y1="10.59993125" x2="53.483" y2="8.99998125" width="0.4" layer="1"/>
 <wire x1="60.083190625" y1="10.5918" x2="60.083190625" y2="10.59993125" width="0.4" layer="16"/>
-<wire x1="49.9872" y1="7.905175" x2="50.85" y2="8.1" width="0.1524" layer="1"/>
-<wire x1="49.9872" y1="7.905175" x2="49.9872" y2="8.99998125" width="0.1524" layer="1"/>
 <wire x1="55.0926" y1="10.5918" x2="55.08295" y2="10.59993125" width="0.1524" layer="1"/>
 <wire x1="55.0926" y1="10.5918" x2="55.083" y2="10.6" width="0.1524" layer="1"/>
@@
 <wire x1="56" y1="9" x2="55.0926" y2="9.9074" width="0.4064" layer="1"/>
 <wire x1="55.0926" y1="9.9074" x2="55.0926" y2="10.5918" width="0.4064" layer="1"/>
+<wire x1="53.483" y1="8.99998125" x2="52.58301875" y2="8.1" width="0.4064" layer="1"/>
+<wire x1="52.58301875" y1="8.1" x2="50.85" y2="8.1" width="0.4064" layer="1"/>
 </signal>
 <signal name="D3">
@@
 <wire x1="72.07351875" y1="41.63491875" x2="72.0852" y2="41.63491875" width="0.4" layer="1"/>
 <wire x1="72.0852" y1="41.63491875" x2="76.09408125" y2="41.63491875" width="0.4" layer="1"/>
-<wire x1="83.95005" y1="8.99998125" x2="83.95005" y2="19.17395" width="0.4" layer="1"/>
+<wire x1="83.95005" y1="8.99998125" x2="83.95005" y2="11" width="0.4" layer="1"/>
+<wire x1="83.95005" y1="11" x2="83.95005" y2="19.17395" width="0.4" layer="1"/>
 <wire x1="83.95005" y1="8.99998125" x2="83.9724" y2="8.99998125" width="0.4" layer="1"/>
 <wire x1="83.9724" y1="8.99998125" x2="87.06688125" y2="8.99998125" width="0.4" layer="1"/>
@@
 <wire x1="93" y1="9" x2="93.667" y2="9.667" width="0.4064" layer="1"/>
 <wire x1="93.667" y1="9.667" x2="93.667" y2="10.6" width="0.4064" layer="1"/>
+<wire x1="88.667" y1="10.6" x2="84.35005" y2="10.6" width="0.4064" layer="1"/>
+<wire x1="84.35005" y1="10.6" x2="83.95005" y2="11" width="0.4064" layer="1"/>
 </signal>
 <signal name="D4">
@@
 <wire x1="31" y1="41" x2="32" y2="41" width="0.4064" layer="1"/>
 <wire x1="32" y1="41" x2="34.187" y2="38.813" width="0.4064" layer="1"/>
-<wire x1="34.187" y1="38.813" x2="34.187" y2="38.187" width="0.4064" layer="1"/>
-<wire x1="34.187" y1="38.187" x2="34.187" y2="37.187" width="0.4064" layer="1"/>
+<wire x1="34.187" y1="38.813" x2="34.187" y2="37.187" width="0.4064" layer="1"/>
 <wire x1="28.375" y1="43.625" x2="31" y2="41" width="0.4064" layer="1"/>
 </signal>
