File: EAGLE/projects/Kontrol_S4_MK4/potboard.sch (EAGLE design)
At the start: 36 parts, among them IC2 74HC595D, IC3 74HC165D

Commit message: update silkscreen
Parts:
- C1, C2: value (none) -> 0.1u
Changed lines of the file:
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@@
 <part name="GND16" library="supply1" library_urn="urn:adsk.eagle:library:371" deviceset="GND" device=""/>
 <part name="GND17" library="supply1" library_urn="urn:adsk.eagle:library:371" deviceset="GND" device=""/>
-<part name="C1" library="adafruit" deviceset="C-US" device="C1206"/>
-<part name="C2" library="adafruit" deviceset="C-US" device="C1206"/>
+<part name="C1" library="adafruit" deviceset="C-US" device="C1206" value="0.1u"/>
+<part name="C2" library="adafruit" deviceset="C-US" device="C1206" value="0.1u"/>
 <part name="R10" library="rcl" library_urn="urn:adsk.eagle:library:334" deviceset="R-US_" device="R0805" package3d_urn="urn:adsk.eagle:package:23553/2" value="82"/>
 <part name="R11" library="rcl" library_urn="urn:adsk.eagle:library:334" deviceset="R-US_" device="R0805" package3d_urn="urn:adsk.eagle:package:23553/2" value="82"/>
