File: KiCAD/Brain C MK5/brain.kicad_pcb (KiCad board)
At the start: 2 copper layers, 143 x 44.8 mm, 20 parts, among them J1 USB_B, J10 Conn_01x10, J11 Conn_01x10, J2 Conn_01x06, J3 Conn_01x10, J4 Conn_01x06, J5 Conn_01x06, J6 Conn_01x06, J7 Conn_01x04, J8 Conn_01x04, J9 Conn_01x10

Commit message: add nect-gen KiCAD files
Parts:
- removed J11: Conn_01x10, Connector_Molex:Molex_PicoBlade_53048-1010_1x10_P1.25mm_Horizontal
- removed J5: Conn_01x06, Connector_Molex:Molex_PicoBlade_53048-0610_1x06_P1.25mm_Horizontal
- removed U$2: TEENSY_LC_ALL_PINS, brain:TEENSY_3.0-3.2&LC_ALL_PINS
- added C1: 100nF, Capacitor_SMD:C_1206_3216Metric_Pad1.33x1.80mm_HandSolder, F.Cu at (118.2, 153.0)
- added C10: 100nF, Capacitor_SMD:C_1206_3216Metric_Pad1.33x1.80mm_HandSolder, F.Cu at (189.2, 113.0)
- added C11: 10uF, Capacitor_SMD:C_1206_3216Metric_Pad1.33x1.80mm_HandSolder, F.Cu at (186.8, 112.9)
- added C12: 2.2nF, Capacitor_SMD:C_1206_3216Metric_Pad1.33x1.80mm_HandSolder, F.Cu at (211.2, 95.8)
- added C13: 100nF, Capacitor_SMD:C_1206_3216Metric_Pad1.33x1.80mm_HandSolder, F.Cu at (136.9, 177.0)
- added C14: 10uF, Capacitor_SMD:C_1206_3216Metric_Pad1.33x1.80mm_HandSolder, F.Cu at (136.9, 180.3)
- added C3: 100nF, Capacitor_SMD:C_1206_3216Metric_Pad1.33x1.80mm_HandSolder, F.Cu at (113.0, 185.8)
- added C5: 10uF, Capacitor_SMD:C_1206_3216Metric_Pad1.33x1.80mm_HandSolder, F.Cu at (112.9, 181.8)
- added C7: 2.2uF, Capacitor_SMD:C_1206_3216Metric_Pad1.33x1.80mm_HandSolder, F.Cu at (193.4, 107.7)
- added C8: 2.2uF, Capacitor_SMD:C_1206_3216Metric_Pad1.33x1.80mm_HandSolder, F.Cu at (193.6, 102.7)
- added C9: 2.2nF, Capacitor_SMD:C_1206_3216Metric_Pad1.33x1.80mm_HandSolder, F.Cu at (187.8, 95.8)
- added R2: 22, Resistor_SMD:R_0805_2012Metric_Pad1.20x1.40mm_HandSolder, F.Cu at (176.8, 105.0)
- added R3: 22, Resistor_SMD:R_0805_2012Metric_Pad1.20x1.40mm_HandSolder, F.Cu at (176.8, 103.0)
- added R4: 22, Resistor_SMD:R_0805_2012Metric_Pad1.20x1.40mm_HandSolder, F.Cu at (176.8, 101.0)
- added R5: 22, Resistor_SMD:R_0805_2012Metric_Pad1.20x1.40mm_HandSolder, F.Cu at (176.8, 99.0)
- added R7: 470, Resistor_SMD:R_0805_2012Metric_Pad1.20x1.40mm_HandSolder, F.Cu at (191.5, 96.8)
- added R8: 470, Resistor_SMD:R_0805_2012Metric_Pad1.20x1.40mm_HandSolder, F.Cu at (207.0, 97.2)
- added U1: Teensy4.0, Teensy:Teensy40_SMT, F.Cu at (137.5, 98.4)
- added U2: LD1117S33TR_SOT223, Package_TO_SOT_SMD:SOT-223-3_TabPin2, F.Cu at (115.5, 145.5)
- added U3: PCM5102, Package_SO:TSSOP-20_4.4x6.5mm_P0.65mm, F.Cu at (185.9, 104.7)
- C2: value 1u -> 10uF
- J2: value Conn_01x06 -> Conn_Coaxial_x2_Isolated; footprint Connector_PinSocket_2.54mm:PinSocket_1x06_P2.54mm_Vertical -> Audio:RCA_double
- J3: value Conn_01x10 -> Conn_01x06; footprint Connector_Molex:Molex_PicoBlade_53048-1010_1x10_P1.25mm_Horizontal -> Connector_Molex:Molex_PicoBlade_53048-0610_1x06_P1.25mm_Horizontal
- J6: value Conn_01x06 -> Conn_01x10; footprint Connector_Molex:Molex_PicoBlade_53048-0610_1x06_P1.25mm_Horizontal -> Connector_Molex:Molex_PicoBlade_53048-1010_1x10_P1.25mm_Horizontal
- J7: value Conn_01x04 -> Conn_01x10; footprint Connector_Molex:Molex_PicoBlade_53048-0410_1x04_P1.25mm_Horizontal -> Connector_Molex:Molex_PicoBlade_53048-1010_1x10_P1.25mm_Horizontal
- J9: value Conn_01x10 -> Conn_01x04; footprint Connector_Molex:Molex_PicoBlade_53048-1010_1x10_P1.25mm_Horizontal -> Connector_Molex:Molex_PicoBlade_53048-0410_1x04_P1.25mm_Horizontal
- R6: value 1M -> 0
- moved C2 99.6 mm to (113.0, 153.0), turned to 90 degrees
- moved J7 80.0 mm to (124.1, 122.0)
- moved J9 52.9 mm to (177.0, 122.0)
- moved J6 36.2 mm to (104.5, 122.0)
- moved J2 30.9 mm to (197.8, 86.2)
- moved R6 28.7 mm to (176.8, 107.7), turned to 0 degrees
- moved JP2 27.4 mm to (170.4, 118.8)
- moved J3 23.9 mm to (140.8, 122.0)
- moved J10 18.1 mm to (87.8, 122.0)
- moved J1 14.3 mm to (174.5, 93.2)
- moved J4 14.2 mm to (164.6, 122.0)
Connections:
- C2 pad 1: /JOG-PRESS-IR -> VDDA
- J1 pad 1: Net-(U$2-PadVIN_PAD) -> unconnected-(J1-VBUS-Pad1)
- J1 pad 2: Net-(U$2-PadD-) -> unconnected-(J1-D--Pad2)
- J1 pad 3: Net-(U$2-PadD+) -> unconnected-(J1-D+-Pad3)
- J10 pad 1: +3.3V -> /595-BRIDGE
- J10 pad 10: /595-LATCH -> /165-BRIDGE
- J10 pad 2: +3.3V -> /595-OUT-MAIN
- J10 pad 3: +3.3V -> /ENCR1
- J10 pad 4: +3.3V -> /ENCR2
- J10 pad 5: +3.3V -> /ENCL1
- J10 pad 6: GND -> /ENCL2
- J10 pad 7: GND -> /CLOCK
- J10 pad 8: GND -> /165-LATCH
- J10 pad 9: /CLOCK -> /CE-595-165
- J2 pad 1: GND -> /PCM5102/AUDIO_OUT_R
- J2 pad 2: +3.3V -> GND
- J2 pad 3: /SDA-EXT -> /PCM5102/AUDIO_OUT_L
- J2 pad 4: /SCL-EXT -> GND
- J3 pad 1: GND -> /POT4
- J3 pad 2: /CLOCK -> /POT3
- J3 pad 3: GND -> /POT2
- J3 pad 4: /MOSI -> /POT1
- J3 pad 5: /SS-SCREEN -> GND
- J4 pad 1: GND -> unconnected-(J4-Pin_1-Pad1)
- J4 pad 2: /CLOCK-EXT -> /JOG-MOVE1
- J4 pad 3: /MISO-EXT -> /JOG-MOVE2
- J4 pad 4: /MOSI-EXT -> GND
- J4 pad 5: /SS-EXT -> Net-(J4-Pin_5)
- J6 pad 1: /POT4 -> +3.3V
- J6 pad 2: /POT3 -> +3.3V
- J6 pad 3: /POT2 -> +3.3V
- J6 pad 4: /POT1 -> +3.3V
- J6 pad 5: GND -> +3.3V
- J6 pad 6: +3.3V -> GND
- J7 pad 1: unconnected-(J7-Pad1) -> +3.3V
- J7 pad 2: /JOG-PRESS-IR -> GND
- J7 pad 3: +3.3V -> /CLOCK
- J7 pad 4: GND -> unconnected-(J7-Pin_4-Pad4)
- J9 pad 1: +3.3V -> unconnected-(J9-Pin_1-Pad1)
- J9 pad 2: GND -> /JOG-PRESS-IR
- J9 pad 3: /CLOCK -> +3.3V
- J9 pad 4: unconnected-(J9-Pad4) -> GND
- JP2 pad 2: Net-(JP2-Pad2) -> Net-(J4-Pin_5)
- R6 pad 1: /JOG-PRESS-IR -> GND
- R6 pad 2: GND -> Net-(U3-FMT)
Routing:
- net /JOG-MOVE2: track 98.8 -> 0.32 mm, vias 2 -> 0
- net /JOG-MOVE1: track 93.9 -> 0.26 mm, vias 2 -> 0
- net /MOSI: track 83.9 -> 0.00 mm
- net /SCL-EXT: track 83.5 -> 0.00 mm
- net /SDA-EXT: track 79.7 -> 0.00 mm
- net /DC-SCREEN: track 69.7 -> 0.00 mm, vias 4 -> 0
- net /CE-595-165: track 93.5 -> 153.4 mm, vias 0 -> 1
- net /595-LATCH: track 59.9 -> 0.00 mm, vias 1 -> 0
- net /JOG-PRESS-IR: track 103.5 -> 45.9 mm
- net /MISO-EXT: track 56.3 -> 0.28 mm, vias 2 -> 0
- net GND: track 0.00 -> 54.8 mm, vias 48 -> 47
- net /595-BRIDGE: track 54.7 -> 0.00 mm, vias 4 -> 0
- net /MOSI-EXT: track 54.3 -> 0.19 mm, vias 2 -> 0
- net /SS-EXT: track 52.9 -> 0.00 mm
- net /CLOCK-EXT: track 51.6 -> 0.00 mm
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Other:
- board text removed: "6. VCC 5. EN 4. GND 3. JOG-2 2. JOG-1 1. NC"
- board text removed: "6. VCC 5. SS 4. MOSI 3. GND 2. CLOCK 1. GND"
- board text removed: "6. VCC 5. SS 4. MOSI 3. MISO 2. CLCK 1. GND"

Commit message: work
Parts:
- removed C5: 10uF, Capacitor_SMD:C_1206_3216Metric_Pad1.33x1.80mm_HandSolder
- removed J10: Conn_01x10, Connector_Molex:Molex_PicoBlade_53048-1010_1x10_P1.25mm_Horizontal
- added C18: 1.2uF, Capacitor_SMD:C_0603_1608Metric, F.Cu at (142.2, 112.2)
- added C19: 1.2uF, Capacitor_SMD:C_0603_1608Metric, F.Cu at (140.5, 112.2)
- added C20: 1.2uF, Capacitor_SMD:C_0603_1608Metric, F.Cu at (144.0, 112.3)
- added C21: 1.2uF, Capacitor_SMD:C_0603_1608Metric, F.Cu at (145.8, 112.3)
- added C22: 1.2uF, Capacitor_SMD:C_0603_1608Metric, F.Cu at (159.0, 116.0)
- added C4: 100nF, Capacitor_SMD:C_0603_1608Metric, F.Cu at (87.9, 172.7)
- added C6: 100nF, Capacitor_SMD:C_0603_1608Metric, F.Cu at (87.9, 175.2)
- added J5: Conn_01x10, Connector_Molex:Molex_PicoBlade_53048-1010_1x10_P1.25mm_Horizontal, F.Cu at (124.4, 122.0)
- added R1: 10R, Resistor_SMD:R_0603_1608Metric, F.Cu at (87.9, 179.8)
- added R13: 2.2K, Resistor_SMD:R_0603_1608Metric, F.Cu at (142.2, 116.6)
- added R14: 2.2K, Resistor_SMD:R_0603_1608Metric, F.Cu at (140.5, 116.6)
- added R15: 2.2K, Resistor_SMD:R_0603_1608Metric, F.Cu at (144.0, 116.6)
- added R16: 2.2K, Resistor_SMD:R_0603_1608Metric, F.Cu at (145.8, 116.6)
- added R17: 2.2K, Resistor_SMD:R_0603_1608Metric, F.Cu at (156.5, 116.8)
- C1, C10, C11, C12, C2, C3, C7, C8, C9: footprint Capacitor_SMD:C_1206_3216Metric_Pad1.33x1.80mm_HandSolder -> Capacitor_SMD:C_0603_1608Metric
- C13: value 100nF -> C_Small; footprint Capacitor_SMD:C_1206_3216Metric_Pad1.33x1.80mm_HandSolder -> Capacitor_SMD:C_0603_1608Metric
- C14: value 10uF -> C_Small; footprint Capacitor_SMD:C_1206_3216Metric_Pad1.33x1.80mm_HandSolder -> Capacitor_SMD:C_0603_1608Metric
- J3, J4: value Conn_01x06 -> Conn_01x10; footprint Connector_Molex:Molex_PicoBlade_53048-0610_1x06_P1.25mm_Horizontal -> Connector_Molex:Molex_PicoBlade_53048-1010_1x10_P1.25mm_Horizontal
- J6: value Conn_01x10 -> Conn_01x06; footprint Connector_Molex:Molex_PicoBlade_53048-1010_1x10_P1.25mm_Horizontal -> Connector_Molex:Molex_PicoBlade_53048-0610_1x06_P1.25mm_Horizontal
- J7: value Conn_01x10 -> Conn_01x04; footprint Connector_Molex:Molex_PicoBlade_53048-1010_1x10_P1.25mm_Horizontal -> Connector_Molex:Molex_PicoBlade_53048-0410_1x04_P1.25mm_Horizontal
- J9: value Conn_01x04 -> Conn_01x06; footprint Connector_Molex:Molex_PicoBlade_53048-0410_1x04_P1.25mm_Horizontal -> Connector_Molex:Molex_PicoBlade_53048-0610_1x06_P1.25mm_Horizontal
- R2, R3, R4, R5, R6, R7, R8: footprint Resistor_SMD:R_0805_2012Metric_Pad1.20x1.40mm_HandSolder -> Resistor_SMD:R_0603_1608Metric
- moved C1 122.0 mm to (234.0, 114.4)
- moved C2 122.0 mm to (228.8, 114.4)
- moved U2 122.0 mm to (231.2, 106.9)
- moved J4 60.2 mm to (104.4, 122.0)
- moved J3 52.9 mm to (87.9, 122.0)
- moved J6 36.6 mm to (141.1, 122.0)
- moved J7 31.2 mm to (155.3, 122.0)
- moved R5 22.7 mm to (197.1, 109.1)
- moved R4 22.5 mm to (197.1, 110.8)
- moved R3 22.4 mm to (197.1, 112.6)
- moved C10 22.3 mm to (209.6, 122.3)
- moved C11 22.3 mm to (207.1, 122.3)
- moved R2 22.3 mm to (197.1, 114.3)
- moved C7 22.3 mm to (213.7, 117.0)
- moved C8 22.3 mm to (213.9, 112.1)
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Connections:
- net /PCM5102/AUDIO_BCLK renamed /DAC (PCM5102)/AUDIO_BCLK
- net /PCM5102/AUDIO_LRCLK renamed /DAC (PCM5102)/AUDIO_LRCLK
- net /PCM5102/AUDIO_MCLK renamed /DAC (PCM5102)/AUDIO_MCLK
- net /PCM5102/AUDIO_TX renamed /DAC (PCM5102)/AUDIO_TX
- net /PCM5102/LDO renamed /DAC (PCM5102)/LDO
- C1 pad 1: +5V -> Net-(U2-VI)
- C10 pad 1: VDDA -> +3.3VA
- C11 pad 1: VDDA -> +3.3VA
- C12 pad 1: /PCM5102/AUDIO_OUT_L -> /DAC (PCM5102)/AUDIO_OUT_L
- C13 pad 1: VDDA -> VBUS
- C14 pad 1: VDDA -> +5V
- C2 pad 1: VDDA -> +3.3VA
- C9 pad 1: /PCM5102/AUDIO_OUT_R -> /DAC (PCM5102)/AUDIO_OUT_R
- J1 pad 1: unconnected-(J1-VBUS-Pad1) -> VBUS
- J1 pad 2: unconnected-(J1-D--Pad2) -> /USB_D-
- J1 pad 3: unconnected-(J1-D+-Pad3) -> /USB_D+
- J3 pad 1: /POT4 -> /Connectors/595_BRIDGE
- J3 pad 2: /POT3 -> /Connectors/595_OUT_MAIN
- J3 pad 3: /POT2 -> /ENCR1
- J3 pad 4: /POT1 -> /ENCR2
- J3 pad 5: GND -> /ENCL1
- J3 pad 6: +3.3V -> /ENCL2
- J4 pad 1: unconnected-(J4-Pin_1-Pad1) -> VCC
- J4 pad 2: /JOG-MOVE1 -> VCC
- J4 pad 3: /JOG-MOVE2 -> VCC
- J4 pad 4: GND -> VCC
- J4 pad 5: Net-(J4-Pin_5) -> VCC
- J4 pad 6: +3.3V -> GND
- J6 pad 1: +3.3V -> /POT_1
- J6 pad 2: +3.3V -> /POT_2
- J6 pad 3: +3.3V -> /POT_3
- J6 pad 4: +3.3V -> /POT_4
- J6 pad 5: +3.3V -> GND
- J6 pad 6: GND -> VCC
- J7 pad 1: +3.3V -> GND
- J7 pad 2: GND -> /FADER_1
- J7 pad 3: /CLOCK -> VCC
- J7 pad 4: unconnected-(J7-Pin_4-Pad4) -> GND
- J8 pad 1: GND -> unconnected-(J8-Pin_1-Pad1)
- J8 pad 2: /POT_VAL -> /JOG_PRESS_IR
- J8 pad 3: +3.3V -> VCC
- J9 pad 2: /JOG-PRESS-IR -> /JOG-MOVE1
- J9 pad 3: +3.3V -> /JOG-MOVE2
- JP1 pad 2: /595-OUT-MAIN -> /Connectors/595_OUT_MAIN
- JP2 pad 1: +3.3V -> VCC
- JP2 pad 2: Net-(J4-Pin_5) -> Net-(J9-Pin_5)
- R7 pad 2: /PCM5102/AUDIO_OUT_R -> /DAC (PCM5102)/AUDIO_OUT_R
- R8 pad 2: /PCM5102/AUDIO_OUT_L -> /DAC (PCM5102)/AUDIO_OUT_L
- U1 pad 1: unconnected-(U1-GND-Pad1) -> GND
- U1 pad 16: unconnected-(U1-3V3-Pad16) -> +3.3V
- U1 pad 2: /MOSI-EXT -> unconnected-(U1-0_RX1_CRX2_CS1-Pad2)
- U1 pad 21: /JOG-PRESS-IR -> /JOG_PRESS_IR
- U1 pad 22: /POT1 -> Net-(U1-15_A1_RX3_SPDIF_IN)
- U1 pad 23: /POT2 -> Net-(U1-16_A2_RX4_SCL1)
- U1 pad 24: /POT3 -> Net-(U1-17_A3_TX4_SDA1)
- U1 pad 25: /POT4 -> Net-(U1-18_A4_SDA0)
- U1 pad 26: /POT_VAL -> Net-(U1-19_A5_SCL0)
- U1 pad 3: /MISO-EXT -> unconnected-(U1-1_TX1_CTX2_MISO1-Pad3)
- U1 pad 31: unconnected-(U1-3V3-Pad31) -> +3.3V
- U1 pad 32: unconnected-(U1-GND-Pad32) -> GND
- U1 pad 33: unconnected-(U1-VIN-Pad33) -> VBUS
- U1 pad 34: unconnected-(U1-VUSB-Pad34) -> VBUS
- U1 pad 53: unconnected-(U1-D--Pad53) -> /USB_D-
- U1 pad 54: unconnected-(U1-D+-Pad54) -> /USB_D+
- U2 pad 2: VDDA -> +3.3VA
- U2 pad 3: +5V -> Net-(U2-VI)
- U3 pad 17: VDDA -> +3.3VA
- U3 pad 8: VDDA -> +3.3VA
Routing:
- net +3.3V: track 196.5 -> 0.00 mm, vias 1 -> 0
- net /CE-595-165: track 153.4 -> 0.00 mm, vias 1 -> 0
- net /165-LATCH: track 124.5 -> 0.00 mm
- net /ENCL2: track 102.1 -> 0.00 mm
- net /ENCL1: track 87.3 -> 0.00 mm
- net /ENCR1: track 83.5 -> 0.00 mm
- net /ENCR2: track 78.2 -> 0.00 mm
- net /CLOCK: track 60.3 -> 0.00 mm
- net GND: track 54.8 -> 0.00 mm, vias 47 -> 0
- net /JOG-PRESS-IR: track 45.9 -> 0.00 mm
- net /165-BRIDGE: track 40.2 -> 0.00 mm, vias 2 -> 0
- net /MISO: track 37.1 -> 0.00 mm, vias 2 -> 0
- net (no net): track 34.4 -> 0.00 mm, vias 1 -> 0
- net /POT_VAL: track 32.2 -> 0.00 mm
- net /POT2: track 27.8 -> 0.00 mm
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Other:
- copper layers 2 -> 4
