File: KiCAD/Brain C MK5/brain.kicad_sch (KiCad schematic)
At the start: 21 parts, among them J1 USB_B, J10 Conn_01x10, J11 Conn_01x10, J12 Conn_Coaxial_x2_Isolated, J2 Conn_01x06, J3 Conn_01x10, J4 Conn_01x06, J5 Conn_01x06, J6 Conn_01x06, J7 Conn_01x04, J8 Conn_01x04, J9 Conn_01x10

Commit message: add nect-gen KiCAD files
Parts:
- removed C2: 1u, Capacitor_SMD:C_1206_3216Metric_Pad1.33x1.80mm_HandSolder, symbol Device:C
- removed J10, J11, J3, J9: Conn_01x10, Connector_Molex:Molex_PicoBlade_53048-1010_1x10_P1.25mm_Horizontal, symbol Connector_Generic:Conn_01x10
- removed J2: Conn_01x06, Connector_PinSocket_2.54mm:PinSocket_1x06_P2.54mm_Vertical, symbol Connector_Generic:Conn_01x06
- removed J4, J5, J6: Conn_01x06, Connector_Molex:Molex_PicoBlade_53048-0610_1x06_P1.25mm_Horizontal, symbol Connector_Generic:Conn_01x06
- removed J7, J8: Conn_01x04, Connector_Molex:Molex_PicoBlade_53048-0410_1x04_P1.25mm_Horizontal, symbol Connector_Generic:Conn_01x04
- removed JP1, JP2: Jumper_2_Bridged, Resistor_SMD:R_0805_2012Metric_Pad1.20x1.40mm_HandSolder, symbol Jumper:Jumper_2_Bridged
- removed R6: 1M, Resistor_SMD:R_0805_2012Metric_Pad1.20x1.40mm_HandSolder, symbol Device:R
- removed U$2: TEENSY_LC_ALL_PINS, brain:TEENSY_3.0-3.2&LC_ALL_PINS, symbol brain-eagle-import:TEENSY_LC_ALL_PINS
- added C15, C5: 10u, symbol Device:C
- added C16: 10uF, symbol Device:C_Small
- added C17: 1.2uF, symbol Device:C_Small
- added R10, R9: 100, symbol Device:R_Small
- added R11: 10R, symbol Device:R_Small
- added R12: 2.2K, symbol Device:R_Small
- added RV1: 10K, symbol Device:R_Potentiometer
- added U1: Teensy4.0, Teensy:Teensy40_SMT, symbol Teensy:Teensy4.0
- renumbered H3 to H2, H2 to H3, J12 to J2
Connections:
- net +3.3V: now also U1.16 (3V3), U1.31 (3V3)
- net 165-LATCH: now also U1.11 (9_OUT1C)
- net 595-LATCH: now also U1.10 (8_TX2_IN1)
- net CE-595-165: now also U1.12 (10_CS_MQSR)
- net CLOCK: now also U1.20 (13_SCK_CRX1_LED)
- net ENCL1: now also U1.4 (2_OUT2)
- net ENCL2: now also U1.5 (3_LRCLK2)
- net ENCR1: now also U1.6 (4_BCLK2)
- net ENCR2: now also U1.7 (5_IN2)
- net GND: now also C15.2, C16.2, C17.1, C5.2, RV1.1, U1.1 (GND), U1.17 (GND), U1.32 (GND)
- net JOG-MOVE1: now also U1.8 (6_OUT1D)
- net JOG-MOVE2: now also U1.9 (7_RX2_OUT1A)
- net MISO: now also U1.14 (12_MISO_MQSL)
- net MISO-EXT: now also U1.3 (1_TX1_CTX2_MISO1)
- net MOSI: now also U1.13 (11_MOSI_CTX1)
- net MOSI-EXT: now also U1.2 (0_RX1_CRX2_CS1)
- net POT1: now also U1.22 (15_A1_RX3_SPDIF_IN)
- net POT2: now also U1.23 (16_A2_RX4_SCL1)
- net POT3: now also U1.24 (17_A3_TX4_SDA1)
- net POT4: now also U1.25 (18_A4_SDA0)
- net VBUS: now reaches J1.1 (VBUS)
- net VBUS: now also U1.33 (VIN), U1.34 (VUSB)
- net USB_D-: now reaches J1.2 (D-)
- net USB_D-: now also U1.53 (D-)
- net USB_D+: now reaches J1.3 (D+)
- net USB_D+: now also U1.54 (D+)
- net DAC (PCM5102)/AUDIO_OUT_R: now reaches J2.1 (In1)
- net GNDA: now reaches J2.2 (Ext1)
- net GNDA: now also J2.4 (Ext2)
- net DAC (PCM5102)/AUDIO_OUT_L: now reaches J2.3 (In2)
- new net: C16.1, R11.1, RV1.3
- new net: R12.1, RV1.2
- new net ADC: C17.2, R12.2
- new net FADER_1: C5.1, R9.2, U1.26 (19_A5_SCL0)
- new net JOG_PRESS_IR: C15.1, R10.2, U1.21 (14_A0_TX3_SPDIF_OUT)
- new net VCC: R11.2
- no-connect marks 10 -> 3
Other:
- added sheet Connectors (connectors.kicad_sch)
- added sheet DAC (PCM5102) (pcm5102.kicad_sch)
- added sheet Power (power.kicad_sch)
- note added: "100R will produce a johnson noise of about 0.19 uV"
- note added: "ESD protection and resistors are built-in the teensy"
- note added: "Filter out high freq noise from fader fc = 160 stolen from NI S4"
- note added: "JUST FOR DEMO"
- note removed: "External SPI"
- note removed: "FX 1"
- note removed: "FX 2"
- note removed: "Fader"
- note removed: "Jog move"
- note removed: "Jog press"
- note removed: "Main 1"
- note removed: "Main 2"
- note removed: "Screen"
- moved on the sheet: J1, J2A, J2B

Commit message: work
Parts:
- removed C15, C5: 10u, symbol Device:C
- removed C16: 10uF, symbol Device:C_Small
- removed C17: 1.2uF, symbol Device:C_Small
- removed R10, R9: 100, symbol Device:R_Small
- removed R11: 10R, symbol Device:R_Small
- removed R12: 2.2K, symbol Device:R_Small
- removed RV1: 10K, symbol Device:R_Potentiometer
- added C18, C19, C20, C21, C22: 1.2uF, Capacitor_SMD:C_0603_1608Metric, symbol Device:C_Small
- added R13, R14, R15, R16, R17: 2.2K, Resistor_SMD:R_0603_1608Metric, symbol Device:R_Small
Connections:
- net FADER_1: now also R17.1; no longer U1.26 (19_A5_SCL0)
- net GND: now also C18.2, C19.2, C20.2, C21.2, C22.2
- net MISO-EXT: no longer names the net of U1.3 (1_TX1_CTX2_MISO1)
- net MOSI-EXT: no longer names the net of U1.2 (0_RX1_CRX2_CS1)
- net POT1: no longer names the net of U1.22 (15_A1_RX3_SPDIF_IN)
- net POT1: now also C19.1, R14.2
- net POT2: no longer names the net of U1.23 (16_A2_RX4_SCL1)
- net POT2: now also C18.1, R13.2
- net POT3: no longer names the net of U1.24 (17_A3_TX4_SDA1)
- net POT3: now also C20.1, R15.2
- net POT4: no longer names the net of U1.25 (18_A4_SDA0)
- net POT4: now also C21.1, R16.2
- new net: C22.1, R17.2, U1.26 (19_A5_SCL0)
- new net POT_1: R14.1
- new net POT_2: R13.1
- new net POT_3: R15.1
- new net POT_4: R16.1
Other:
- sheet Connectors ports: added 165_LATCH, 595_LATCH, CE_595_165, CLOCK, ENC_L1, ENC_L2, ENC_R1, ENC_R2, FADER_1, JOG_MOVE_1, JOG_MOVE_2, JOG_PRESS_IR, MISO, MOSI, POT_1, POT_2, POT_3, POT_4; removed none
- note added: "Fc = 60Hz Step response = 0.01s Johnson noise Vn(RMS) = 0.872108 uV"
- note removed: "100R will produce a johnson noise of about 0.19 uV"
- note removed: "Filter out high freq noise from fader fc = 160 stolen from NI S4"
- note removed: "JUST FOR DEMO"
- moved on the sheet: H1, H2, H3, H4
