File: KiCAD/Brain C MK5/pcm5102.kicad_sch (KiCad schematic)
At the start: 17 parts, among them U3 PCM5102

Commit message: work
Parts:
- C10, C11, C12, C3, C4, C6, C7, C8, C9: footprint Capacitor_SMD:C_1206_3216Metric_Pad1.33x1.80mm_HandSolder -> Capacitor_SMD:C_0603_1608Metric
- R2, R3, R4, R5, R6, R7, R8: footprint Resistor_SMD:R_0805_2012Metric_Pad1.20x1.40mm_HandSolder -> Resistor_SMD:R_0603_1608Metric
Changed lines of the file:
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@@
       (effects (font (size 1.27 1.27)))
     )
-    (property "Footprint" "Resistor_SMD:R_0805_2012Metric_Pad1.20x1.40mm_HandSolder" (at 125.73 56.515 0)
+    (property "Footprint" "Resistor_SMD:R_0603_1608Metric" (at 125.73 56.515 0)
       (effects (font (size 1.27 1.27)) hide)
     )
@@
       (effects (font (size 1.27 1.27)) (justify left))
     )
-    (property "Footprint" "Capacitor_SMD:C_1206_3216Metric_Pad1.33x1.80mm_HandSolder" (at 59.69 43.815 0)
+    (property "Footprint" "Capacitor_SMD:C_0603_1608Metric" (at 59.69 43.815 0)
       (effects (font (size 1.27 1.27)) hide)
     )
@@
       (effects (font (size 1.27 1.27)) (justify left))
     )
-    (property "Footprint" "Capacitor_SMD:C_1206_3216Metric_Pad1.33x1.80mm_HandSolder" (at 95.885 67.945 0)
+    (property "Footprint" "Capacitor_SMD:C_0603_1608Metric" (at 95.885 67.945 0)
       (effects (font (size 1.27 1.27)) hide)
     )
@@
       (effects (font (size 1.27 1.27)) (justify left))
     )
-    (property "Footprint" "Capacitor_SMD:C_1206_3216Metric_Pad1.33x1.80mm_HandSolder" (at 99.695 27.94 0)
+    (property "Footprint" "Capacitor_SMD:C_0603_1608Metric" (at 99.695 27.94 0)
       (effects (font (size 1.27 1.27)) hide)
     )
@@
       (effects (font (size 1.27 1.27)) (justify left))
     )
-    (property "Footprint" "Capacitor_SMD:C_1206_3216Metric_Pad1.33x1.80mm_HandSolder" (at 128.27 60.96 0)
+    (property "Footprint" "Capacitor_SMD:C_0603_1608Metric" (at 128.27 60.96 0)
       (effects (font (size 1.27 1.27)) hide)
     )
@@
       (effects (font (size 1.27 1.27)))
     )
-    (property "Footprint" "Resistor_SMD:R_0805_2012Metric_Pad1.20x1.40mm_HandSolder" (at 67.945 64.135 0)
+    (property "Footprint" "Resistor_SMD:R_0603_1608Metric" (at 67.945 64.135 0)
       (effects (font (size 1.27 1.27)) hide)
     )
@@
       (effects (font (size 1.27 1.27)))
     )
-    (property "Footprint" "Resistor_SMD:R_0805_2012Metric_Pad1.20x1.40mm_HandSolder" (at 67.945 56.515 0)
+    (property "Footprint" "Resistor_SMD:R_0603_1608Metric" (at 67.945 56.515 0)
       (effects (font (size 1.27 1.27)) hide)
     )
@@
       (effects (font (size 1.27 1.27)))
     )
-    (property "Footprint" "Resistor_SMD:R_0805_2012Metric_Pad1.20x1.40mm_HandSolder" (at 67.945 59.055 0)
+    (property "Footprint" "Resistor_SMD:R_0603_1608Metric" (at 67.945 59.055 0)
       (effects (font (size 1.27 1.27)) hide)
     )
@@
       (effects (font (size 1.27 1.27)) (justify right))
     )
-    (property "Footprint" "Resistor_SMD:R_0805_2012Metric_Pad1.20x1.40mm_HandSolder" (at 64.135 79.375 0)
+    (property "Footprint" "Resistor_SMD:R_0603_1608Metric" (at 64.135 79.375 0)
       (effects (font (size 1.27 1.27)) hide)
     )
@@
       (effects (font (size 1.27 1.27)) (justify left))
     )
-    (property "Footprint" "Capacitor_SMD:C_1206_3216Metric_Pad1.33x1.80mm_HandSolder" (at 109.855 27.94 0)
+    (property "Footprint" "Capacitor_SMD:C_0603_1608Metric" (at 109.855 27.94 0)
       (effects (font (size 1.27 1.27)) hide)
     )
@@
       (effects (font (size 1.27 1.27)) (justify left))
     )
-    (property "Footprint" "Capacitor_SMD:C_1206_3216Metric_Pad1.33x1.80mm_HandSolder" (at 114.935 79.375 0)
+    (property "Footprint" "Capacitor_SMD:C_0603_1608Metric" (at 114.935 79.375 0)
       (effects (font (size 1.27 1.27)) hide)
     )
@@
       (effects (font (size 1.27 1.27)))
     )
-    (property "Footprint" "Resistor_SMD:R_0805_2012Metric_Pad1.20x1.40mm_HandSolder" (at 104.775 59.055 0)
+    (property "Footprint" "Resistor_SMD:R_0603_1608Metric" (at 104.775 59.055 0)
       (effects (font (size 1.27 1.27)) hide)
     )
@@
       (effects (font (size 1.27 1.27)) (justify left))
     )
-    (property "Footprint" "Capacitor_SMD:C_1206_3216Metric_Pad1.33x1.80mm_HandSolder" (at 107.315 63.5 0)
+    (property "Footprint" "Capacitor_SMD:C_0603_1608Metric" (at 107.315 63.5 0)
       (effects (font (size 1.27 1.27)) hide)
     )
@@
       (effects (font (size 1.27 1.27)) (justify left))
     )
-    (property "Footprint" "Capacitor_SMD:C_1206_3216Metric_Pad1.33x1.80mm_HandSolder" (at 59.69 27.94 0)
+    (property "Footprint" "Capacitor_SMD:C_0603_1608Metric" (at 59.69 27.94 0)
       (effects (font (size 1.27 1.27)) hide)
     )
@@
       (effects (font (size 1.27 1.27)) (justify left))
     )
-    (property "Footprint" "Capacitor_SMD:C_1206_3216Metric_Pad1.33x1.80mm_HandSolder" (at 101.6 81.915 0)
+    (property "Footprint" "Capacitor_SMD:C_0603_1608Metric" (at 101.6 81.915 0)
       (effects (font (size 1.27 1.27)) hide)
     )
@@
       (effects (font (size 1.27 1.27)))
     )
-    (property "Footprint" "Resistor_SMD:R_0805_2012Metric_Pad1.20x1.40mm_HandSolder" (at 67.945 61.595 0)
-      (effects (font (size 1.27 1.27)) hide)
-    )
+    (property "Footprint" "Resistor_SMD:R_0603_1608Metric" (at 67.945 61.595 0)
+      (effects (font (size 1.27 1.27)) hide)
+    )
