File: KiCAD/Brain C MK5/power.kicad_sch (KiCad schematic)
At the start: 7 parts, among them U2 LD1117S33TR_SOT223

Commit message: work
Parts:
- C1, C2: footprint Capacitor_SMD:C_1206_3216Metric_Pad1.33x1.80mm_HandSolder -> Capacitor_SMD:C_0603_1608Metric
- C13, C14: footprint (none) -> Capacitor_SMD:C_0603_1608Metric
- R1: footprint (none) -> Resistor_SMD:R_0603_1608Metric
Changed lines of the file:
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@@
       (effects (font (size 1.27 1.27)) (justify left))
     )
-    (property "Footprint" "" (at 73.025 60.96 0)
+    (property "Footprint" "Capacitor_SMD:C_0603_1608Metric" (at 73.025 60.96 0)
       (effects (font (size 1.27 1.27)) hide)
     )
@@
       (effects (font (size 1.27 1.27)) (justify left))
     )
-    (property "Footprint" "Capacitor_SMD:C_1206_3216Metric_Pad1.33x1.80mm_HandSolder" (at 119.38 58.42 0)
+    (property "Footprint" "Capacitor_SMD:C_0603_1608Metric" (at 119.38 58.42 0)
       (effects (font (size 1.27 1.27)) hide)
     )
@@
       (effects (font (size 1.27 1.27)))
     )
-    (property "Footprint" "" (at 89.535 57.658 90)
+    (property "Footprint" "Resistor_SMD:R_0603_1608Metric" (at 89.535 57.658 90)
       (effects (font (size 1.27 1.27)) hide)
     )
@@
       (effects (font (size 1.27 1.27)) (justify left))
     )
-    (property "Footprint" "Capacitor_SMD:C_1206_3216Metric_Pad1.33x1.80mm_HandSolder" (at 96.52 58.42 0)
+    (property "Footprint" "Capacitor_SMD:C_0603_1608Metric" (at 96.52 58.42 0)
       (effects (font (size 1.27 1.27)) hide)
     )
@@
       (effects (font (size 1.27 1.27)) (justify left))
     )
-    (property "Footprint" "" (at 56.515 60.96 0)
-      (effects (font (size 1.27 1.27)) hide)
-    )
+    (property "Footprint" "Capacitor_SMD:C_0603_1608Metric" (at 56.515 60.96 0)
+      (effects (font (size 1.27 1.27)) hide)
+    )
